File: Harvware/VALDIKLIS_v2.0_DIN.brd (EAGLE design)
At the start: 100 x 86.4 mm, 45 parts, among them IC1 ATMEGA1284, K1 G5V1, K2 G5V1, K3 G5V1, K4 G5V1, T2 TIP120, T3 TIP120, X12 12MHZ, Y2 16MHz

Commit message: tesinys
Parts:
- removed T2, T3: TIP120, rocketfarm:TO220AH
- added Q3, Q4: TIP120V, rocketfarm:TO220AV
- added R9: (no value), resistor-1:0309V
- R7: value 2k2 -> 10k; device resistor-1:0207/10 -> SteveMarple:RES-AXIAL-0.4
- R8: value 2k2 -> (none); device resistor-1:0207/10 -> resistor-1:0309V
- moved R6 92.4 mm to (43.8, 31.8), turned to 270 degrees
- moved R5 84.6 mm to (37.5, 31.8), turned to 270 degrees
- moved R4 76.9 mm to (31.1, 31.8), turned to 270 degrees
- moved R3 69.2 mm to (24.8, 31.8), turned to 270 degrees
- moved R7 25.0 mm to (52.1, 64.8), turned to 90 degrees
- moved K1 15.1 mm to (84.5, 8.26), turned to 0 degrees
- moved IC2 11.3 mm to (67.3, 36.2)
- moved K2 6.38 mm to (73.7, 21.0)
- moved R8 5.75 mm to (81.9, 69.2), turned to 90 degrees
- moved K3 5.75 mm to (62.9, 21.0)
- moved K4 5.12 mm to (52.1, 21.0)
- renumbered U$11 to U$3, U$12 to U$1, U$13 to U$2, U$17 to U$5, U$19 to U$4
Connections:
- removed net GND2: T2.E, T3.E
- new net N$21: SSR3.DS2, U$7.3
- new net N$22: SSR3.DS1, U$7.4
- new net N$23: SSR4.DS1, U$7.2
- new net N$24: SSR4.DS2, U$7.1
- new net N$25: SSR5.DS1, U$9.4
- new net N$26: SSR5.DS2, U$9.3
- new net N$27: SSR6.DS1, U$9.2
- new net N$28: SSR6.DS2, U$9.1
- new net N$29: R1.1
- new net N$30: R2.1
- new net N$31: R3.2, SSR3.A
- new net N$32: R3.1
- new net N$33: R4.2, SSR4.A
- new net N$34: R4.1
- new net N$35: R5.1
- new net N$36: R5.2, SSR5.A
- new net N$37: R6.1
- new net N$39: R6.2, SSR6.A
- new net N$41: R8.1
- net D6: no longer R7.1
- net D9: now also R9.1; no longer R8.1
- net GND: now also Q3.E, Q4.E, SSR1.K, SSR2.K, SSR3.K, SSR4.K, SSR5.K, SSR6.K, U$4.1, U$4.3
- net N$13: now also Q3.B, R8.2; no longer T2.C
- net N$14: now also Q4.B, R9.2; no longer T3.C
- net N$7: now also Q4.C, U$4.2; no longer R8.2, T3.B
- net N$8: now also Q3.C, U$4.4; no longer R7.2, T2.B
