File: Harvware/VALDIKLIS_v2.0_DIN.sch (EAGLE design)
At the start: 27 parts, among them IC4 ATMEGA1284, K1 G5V1, K2 G5V1, K3 G5V1, K4 G5V1, X12 12MHZ

Commit message: pradžia 2
Parts:
- removed IC4: ATMEGA1284, SteveMarple:ATMEGA644-20PU
- removed U$1, U$2, U$3, U$4, U$5, U$8: S202T02, relay-1:S202T02
- added C10, C11: 22p, SparkFun:CAPPTH
- added C5, C7, C9: 100n, SparkFun:CAPPTH
- added C6: 4u7, SparkFun:CAP_POLPTH2
- added IC1: ATMEGA1284, SteveMarple:ATMEGA644-20PU
- added L1: 10uH, SteveMarple:INDUCTOR0.4"-AXIAL
- added R1, R2, R3, R4, R5, R6: (no value), resistor-1:R-EU_0309/V
- added R7, R8: 2k2, resistor-1:R-US_0207/10
- added SSR1, SSR2, SSR3, SSR4, SSR5, SSR6: S202T02, relay-1:S202T02
- added T2, T3: TIP120, rocketfarm:TIP120
- added Y2: 16MHz, SteveMarple:CRYSTAL-RESONATOR
Connections:
- removed net 10: IC4.PCINT12/OC0B/SS_PB4
- removed net 14: IC4.PCINT23/TOSC2_PC7
- removed net 15: IC4.PCINT22/TOSC1_PC6
- removed net 22: IC4.PCINT28/OC1B_PD4
- removed net 23: IC4.PCINT31/OC2A_PD7
- removed net 4: IC4.PCINT8/XCK0/T0_PB0
- removed net 5: IC4.PCINT9/CLKO/T1_PB1
- removed net 6: IC4.PCINT10/INT2/AIN0_PB2
- removed net 7: IC4.PCINT11/OC0A/AIN1_PB3
- removed net 8: IC4.PCINT30/OC2B/ICP_PD6
- removed net 9: IC4.PCINT29/OC1A_PD5
- removed net AVCC1: IC4.AVCC
- removed net GND1: IC4.GND, IC4.GND@1
- removed net VCC1: IC4.VCC
- new net AVCC: C9.1, IC1.AVCC, L1.1
- new net D10: IC1.PCINT12/OC0B/SS_PB4
- new net D14: IC1.PCINT23/TOSC2_PC7
- new net D15: IC1.PCINT22/TOSC1_PC6
- new net D22: IC1.PCINT28/OC1B_PD4
- new net D23: IC1.PCINT31/OC2A_PD7
- new net D4: IC1.PCINT8/XCK0/T0_PB0
- new net D5: IC1.PCINT9/CLKO/T1_PB1
- new net D6: IC1.PCINT10/INT2/AIN0_PB2, R7.1
- new net D7: IC1.PCINT11/OC0A/AIN1_PB3
- new net D8: IC1.PCINT30/OC2B/ICP_PD6
- new net D9: IC1.PCINT29/OC1A_PD5, R8.1
- new net GND2: T2.E, T3.E
- new net N$13: T2.C
- new net N$14: T3.C
- new net N$16: C11.1, IC1.XTAL1, Y2.3
- new net N$17: C10.1, IC1.XTAL2, Y2.1
- new net N$18: R1.2, SSR1.A
- new net N$19: SSR2.DS1, U$62.K
- new net N$20: R2.2, SSR2.A
- new net N$6: SSR1.DS2, U$63.K
- new net N$7: R8.2, T3.B
- new net N$8: R7.2, T2.B
- new net VCC: C6.+, C7.1, IC1.VCC, L1.2
- net !RESET: now also IC1.!RESET; no longer IC4.!RESET
- net 0(RX0): now also IC1.PCINT24/RXD0_PD0; no longer IC4.PCINT24/RXD0_PD0
- net 1(TX0): now also IC1.PCINT25/TXD0_PD1; no longer IC4.PCINT25/TXD0_PD1
- net 11(MOSI): now also IC1.PCINT13/MOSI_PB5; no longer IC4.PCINT13/MOSI_PB5
- net 12(MISO): now also IC1.PCINT14/MISO_PB6; no longer IC4.PCINT14/MISO_PB6
- net 13(SCK): now also IC1.PCINT15/SCK_PB7; no longer IC4.PCINT15/SCK_PB7
- net 16(TDI): now also IC1.PCINT21/TDI_PC5; no longer IC4.PCINT21/TDI_PC5
- net 17(TDO): now also IC1.PCINT20/TDO_PC4; no longer IC4.PCINT20/TDO_PC4
- net 18(TMS): now also IC1.PCINT19/TMS_PC3; no longer IC4.PCINT19/TMS_PC3
- net 19(TCK): now also IC1.PCINT18/TCK_PC2; no longer IC4.PCINT18/TCK_PC2
- net 2(RX1): now also IC1.PCINT26/INT0_PD2; no longer IC4.PCINT26/INT0_PD2
- net 20(SDA): now also IC1.PCINT17/SDA_PC1; no longer IC4.PCINT17/SDA_PC1
- net 21(SCL): now also IC1.PCINT16/SCL_PC0; no longer IC4.PCINT16/SCL_PC0
- net 3(TX1): now also IC1.PCINT27/INT1_PD3; no longer IC4.PCINT27/INT1_PD3
- net A0: now also IC1.PCINT7/ADC7_PA7; no longer IC4.PCINT7/ADC7_PA7
- net A1: now also IC1.PCINT6/ADC6_PA6; no longer IC4.PCINT6/ADC6_PA6
- net A2: now also IC1.PCINT5/ADC5_PA5; no longer IC4.PCINT5/ADC5_PA5
- net A3: now also IC1.PCINT4/ADC4_PA4; no longer IC4.PCINT4/ADC4_PA4
- net A4: now also IC1.PCINT3/ADC3_PA3; no longer IC4.PCINT3/ADC3_PA3
- net A5: now also IC1.PCINT2/ADC2_PA2; no longer IC4.PCINT2/ADC2_PA2
- net A6: now also IC1.PCINT1/ADC1_PA1; no longer IC4.PCINT1/ADC1_PA1
- net A7: now also IC1.PCINT0/ADC0_PA0; no longer IC4.PCINT0/ADC0_PA0
- net AREF: now also C5.1, IC1.AREF; no longer IC4.AREF
- net GND: now also C10.2, C11.2, C5.2, C6.-, C7.2, C9.2, IC1.GND, IC1.GND@1, Y2.2
- net N$10: now also SSR2.DS2, U$61.K; no longer IC4.XTAL2
- net N$9: now also SSR1.DS1, U$64.K; no longer IC4.XTAL1
Other:
- note added: "Omit load capacitors if resonator"
- note added: "fitted instead of crystal"
- moved on the sheet: U$61, U$62, U$63, U$64

Commit message: tesinys
Parts:
- removed T2, T3: TIP120, rocketfarm:TIP120
- removed U$19: 4-3.50, con-phoenix-350-1:4-3.50
- added Q3, Q4: TIP120V, rocketfarm:TIP120V
- added R9: (no value), resistor-1:R-EU_0309/V
- added U$4: 4-3.50, con-phoenix-350-1:4-3.50
- R7: value 2k2 -> 10k; device resistor-1:R-US_0207/10 -> SteveMarple:RESISTOR
- R8: value 2k2 -> (none); device resistor-1:R-US_0207/10 -> resistor-1:R-EU_0309/V
- renumbered U$11 to U$3, U$12 to U$1, U$13 to U$2, U$17 to U$5
Connections:
- removed net GND2: T2.E, T3.E
- new net N$21: SSR3.DS2, U$73.K
- new net N$22: SSR3.DS1, U$74.K
- new net N$23: SSR4.DS1, U$72.K
- new net N$24: SSR4.DS2, U$71.K
- new net N$25: SSR5.DS1, U$94.K
- new net N$26: SSR5.DS2, U$93.K
- new net N$27: SSR6.DS1, U$92.K
- new net N$28: SSR6.DS2, U$91.K
- new net N$29: R1.1
- new net N$30: R2.1
- new net N$31: R3.2, SSR3.A
- new net N$32: R3.1
- new net N$33: R4.2, SSR4.A
- new net N$34: R4.1
- new net N$35: R5.1
- new net N$36: R5.2, SSR5.A
- new net N$37: R6.1
- new net N$39: R6.2, SSR6.A
- new net N$41: R8.1
- net D6: no longer R7.1
- net D9: now also R9.1; no longer R8.1
- net GND: now also Q3.E, Q4.E, SSR1.K, SSR2.K, SSR3.K, SSR4.K, SSR5.K, SSR6.K, U$41.K, U$43.K
- net N$13: now also Q3.B, R8.2; no longer T2.C
- net N$14: now also Q4.B, R9.2; no longer T3.C
- net N$7: now also Q4.C, U$42.K; no longer R8.2, T3.B
- net N$8: now also Q3.C, U$44.K; no longer R7.2, T2.B
Other:
- moved on the sheet: R1, R2, R3, R4, R5, R6, SSR1, SSR2, SSR3, SSR4, SSR5, SSR6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
