File: Harvware/VALDIKLIS_v2.0_DIN.sch (EAGLE design)
At the start: 56 parts, among them IC1 ATMEGA1284, J1 6-3.50, J10 6-3.50, J2 6-3.50, J3 6-3.50, J4 4-3.50, J5 2-3.50, J6 4-3.50, J7 4-3.50, J8 4-3.50, J9 6-3.50, K1 G5V1, K2 G5V1, K3 G5V1, K4 G5V1, Q3 TIP120V, Q4 TIP120V, X12 12MHZ, Y2 16MHz

Commit message: 1
Connections:
- net 0(RX0) renamed D8(RX0)
- net 1(TX0) renamed D9(TX0)
- net 11(MOSI) renamed D5(MOSI)
- net 12(MISO) renamed D6(MISO)
- net 13(SCK) renamed D7(SCK)
- net 16(TDI) renamed D21(TDI)
- net 17(TDO) renamed D20(TDO)
- net 18(TMS) renamed D19(TMS)
- net 19(TCK) renamed D18(TCK)
- net 2(RX1) renamed D10(RX1)
- net 20(SDA) renamed D17(SDA)
- net 21(SCL) renamed D16(SCL)
- net 3(TX1) renamed D11(TX1)
- net A0 renamed A7(31)
- net A1 renamed A6(30)
- net A2 renamed A5(29)
- net A3 renamed A4(28)
- net A4 renamed A3(27)
- net A5 renamed A2(26)
- net A6 renamed A1(25)
- net A7 renamed A0(24)
- net D5 renamed D1
- net D6 renamed D2
- net D7 renamed D3
- removed net D10: IC1.PCINT12/OC0B/SS_PB4
- removed net D8: IC1.PCINT30/OC2B/ICP_PD6
- new net D0: IC1.PCINT8/XCK0/T0_PB0
- new net D12: IC1.PCINT28/OC1B_PD4
- new net D13: IC1.PCINT29/OC1A_PD5
- net D14: now also IC1.PCINT30/OC2B/ICP_PD6; no longer IC1.PCINT23/TOSC2_PC7
- net D15: now also IC1.PCINT31/OC2A_PD7; no longer IC1.PCINT22/TOSC1_PC6
- net D22: now also IC1.PCINT22/TOSC1_PC6; no longer IC1.PCINT28/OC1B_PD4
- net D23: now also IC1.PCINT23/TOSC2_PC7; no longer IC1.PCINT31/OC2A_PD7
- net D4: now also IC1.PCINT12/OC0B/SS_PB4; no longer IC1.PCINT8/XCK0/T0_PB0
- net D9: no longer IC1.PCINT29/OC1A_PD5
Changed lines of the file:
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@@
 <setting verticaltext="up"/>
 </settings>
-<grid distance="1.27" unitdist="mm" unit="mm" style="lines" multiple="1" display="no" altdistance="0.01" altunitdist="inch" altunit="mm"/>
+<grid distance="0.1" unitdist="inch" unit="inch" style="lines" multiple="1" display="no" altdistance="0.01" altunitdist="inch" altunit="inch"/>
 <layers>
 <layer number="1" name="Top" color="4" fill="1" visible="no" active="no"/>
@@
 </segment>
 </net>
-<net name="13(SCK)" class="0">
+<net name="D7(SCK)" class="0">
 <segment>
 <wire x1="195.58" y1="223.52" x2="187.96" y2="223.52" width="0.1524" layer="91"/>
@@
 </segment>
 </net>
-<net name="20(SDA)" class="0">
+<net name="D17(SDA)" class="0">
 <segment>
 <wire x1="256.54" y1="198.12" x2="259.08" y2="198.12" width="0.1524" layer="91"/>
@@
 </segment>
 </net>
-<net name="21(SCL)" class="0">
+<net name="D16(SCL)" class="0">
 <segment>
 <wire x1="256.54" y1="195.58" x2="259.08" y2="195.58" width="0.1524" layer="91"/>
@@
 </segment>
 </net>
-<net name="A4" class="0">
+<net name="A3(27)" class="0">
 <segment>
 <wire x1="256.54" y1="233.68" x2="259.08" y2="233.68" width="0.1524" layer="91"/>
@@
 </segment>
 </net>
-<net name="A5" class="0">
+<net name="A2(26)" class="0">
 <segment>
 <wire x1="256.54" y1="236.22" x2="259.08" y2="236.22" width="0.1524" layer="91"/>
@@
 </segment>
 </net>
-<net name="A0" class="0">
+<net name="A7(31)" class="0">
 <segment>
 <wire x1="256.54" y1="223.52" x2="259.08" y2="223.52" width="0.1524" layer="91"/>
@@
 </segment>
 </net>
-<net name="A1" class="0">
+<net name="A6(30)" class="0">
 <segment>
 <wire x1="256.54" y1="226.06" x2="259.08" y2="226.06" width="0.1524" layer="91"/>
@@
 </segment>
 </net>
-<net name="A2" class="0">
+<net name="A5(29)" class="0">
 <segment>
 <wire x1="256.54" y1="228.6" x2="259.08" y2="228.6" width="0.1524" layer="91"/>
@@
 </segment>
 </net>
-<net name="A3" class="0">
+<net name="A4(28)" class="0">
 <segment>
 <wire x1="256.54" y1="231.14" x2="259.08" y2="231.14" width="0.1524" layer="91"/>
@@
 </segment>
 </net>
-<net name="A6" class="0">
+<net name="A1(25)" class="0">
 <segment>
 <wire x1="256.54" y1="238.76" x2="259.08" y2="238.76" width="0.1524" layer="91"/>
@@
 </segment>
 </net>
-<net name="A7" class="0">
+<net name="A0(24)" class="0">
 <segment>
 <wire x1="256.54" y1="241.3" x2="259.08" y2="241.3" width="0.1524" layer="91"/>
@@
 </segment>
 </net>
-<net name="11(MOSI)" class="0">
+<net name="D5(MOSI)" class="0">
 <segment>
 <wire x1="195.58" y1="228.6" x2="187.96" y2="228.6" width="0.1524" layer="91"/>
@@
 </segment>
 </net>
-<net name="12(MISO)" class="0">
+<net name="D6(MISO)" class="0">
 <segment>
 <wire x1="195.58" y1="226.06" x2="187.96" y2="226.06" width="0.1524" layer="91"/>
@@
 </segment>
 </net>
-<net name="1(TX0)" class="0">
+<net name="D9(TX0)" class="0">
 <segment>
 <wire x1="195.58" y1="205.74" x2="187.96" y2="205.74" width="0.1524" layer="91"/>
@@
 </segment>
 </net>
-<net name="3(TX1)" class="0">
+<net name="D11(TX1)" class="0">
 <segment>
 <wire x1="195.58" y1="200.66" x2="187.96" y2="200.66" width="0.1524" layer="91"/>
@@
 </segment>
 </net>
-<net name="0(RX0)" class="0">
+<net name="D8(RX0)" class="0">
 <segment>
 <wire x1="195.58" y1="208.28" x2="187.96" y2="208.28" width="0.1524" layer="91"/>
@@
 </segment>
 </net>
-<net name="2(RX1)" class="0">
+<net name="D10(RX1)" class="0">
 <segment>
 <wire x1="195.58" y1="203.2" x2="187.96" y2="203.2" width="0.1524" layer="91"/>
@@
 </segment>
 </net>
-<net name="D22" class="0">
+<net name="D12" class="0">
 <segment>
 <wire x1="195.58" y1="198.12" x2="187.96" y2="198.12" width="0.1524" layer="91"/>
@@
 </segment>
 </net>
-<net name="D8" class="0">
+<net name="D0" class="0">
+<segment>
+<wire x1="195.58" y1="241.3" x2="187.96" y2="241.3" width="0.1524" layer="91"/>
+<label x="185.42" y="241.3" size="1.778" layer="95" rot="MR0"/>
+<pinref part="IC1" gate="G$1" pin="PCINT8/XCK0/T0_PB0"/>
+</segment>
+</net>
+<net name="D1" class="0">
+<segment>
+<wire x1="195.58" y1="238.76" x2="187.96" y2="238.76" width="0.1524" layer="91"/>
+<label x="185.42" y="238.76" size="1.778" layer="95" rot="MR0"/>
+<pinref part="IC1" gate="G$1" pin="PCINT9/CLKO/T1_PB1"/>
+</segment>
+</net>
+<net name="D3" class="0">
+<segment>
+<wire x1="195.58" y1="233.68" x2="187.96" y2="233.68" width="0.1524" layer="91"/>
+<label x="185.42" y="233.68" size="1.778" layer="95" rot="MR0"/>
+<pinref part="IC1" gate="G$1" pin="PCINT11/OC0A/AIN1_PB3"/>
+</segment>
+</net>
+<net name="D4" class="0">
+<segment>
+<wire x1="195.58" y1="231.14" x2="187.96" y2="231.14" width="0.1524" layer="91"/>
+<label x="185.42" y="231.14" size="1.778" layer="95" rot="MR0"/>
+<pinref part="IC1" gate="G$1" pin="PCINT12/OC0B/SS_PB4"/>
+</segment>
+</net>
+<net name="D14" class="0">
 <segment>
 <wire x1="195.58" y1="193.04" x2="187.96" y2="193.04" width="0.1524" layer="91"/>
@@
 </segment>
 </net>
-<net name="D4" class="0">
-<segment>
-<wire x1="195.58" y1="241.3" x2="187.96" y2="241.3" width="0.1524" layer="91"/>
-<label x="185.42" y="241.3" size="1.778" layer="95" rot="MR0"/>
-<pinref part="IC1" gate="G$1" pin="PCINT8/XCK0/T0_PB0"/>
-</segment>
-</net>
-<net name="D5" class="0">
-<segment>
-<wire x1="195.58" y1="238.76" x2="187.96" y2="238.76" width="0.1524" layer="91"/>
-<label x="185.42" y="238.76" size="1.778" layer="95" rot="MR0"/>
-<pinref part="IC1" gate="G$1" pin="PCINT9/CLKO/T1_PB1"/>
-</segment>
-</net>
-<net name="D7" class="0">
-<segment>
-<wire x1="195.58" y1="233.68" x2="187.96" y2="233.68" width="0.1524" layer="91"/>
-<label x="185.42" y="233.68" size="1.778" layer="95" rot="MR0"/>
-<pinref part="IC1" gate="G$1" pin="PCINT11/OC0A/AIN1_PB3"/>
-</segment>
-</net>
-<net name="D10" class="0">
-<segment>
-<wire x1="195.58" y1="231.14" x2="187.96" y2="231.14" width="0.1524" layer="91"/>
-<label x="185.42" y="231.14" size="1.778" layer="95" rot="MR0"/>
-<pinref part="IC1" gate="G$1" pin="PCINT12/OC0B/SS_PB4"/>
-</segment>
-</net>
-<net name="D14" class="0">
-<segment>
-<wire x1="256.54" y1="213.36" x2="259.08" y2="213.36" width="0.1524" layer="91"/>
-<label x="261.62" y="213.36" size="1.778" layer="95"/>
-<pinref part="IC1" gate="G$1" pin="PCINT23/TOSC2_PC7"/>
-</segment>
-</net>
 <net name="D15" class="0">
 <segment>
-<wire x1="256.54" y1="210.82" x2="259.08" y2="210.82" width="0.1524" layer="91"/>
-<label x="261.62" y="210.82" size="1.778" layer="95"/>
-<pinref part="IC1" gate="G$1" pin="PCINT22/TOSC1_PC6"/>
-</segment>
-</net>
-<net name="16(TDI)" class="0">
+<wire x1="256.54" y1="193.04" x2="259.08" y2="193.04" width="0.1524" layer="91"/>
+<label x="261.62" y="193.04" size="1.778" layer="95"/>
+<pinref part="IC1" gate="G$1" pin="PCINT31/OC2A_PD7"/>
+</segment>
+</net>
+<net name="D21(TDI)" class="0">
 <segment>
 <wire x1="256.54" y1="208.28" x2="259.08" y2="208.28" width="0.1524" layer="91"/>
@@
 </segment>
 </net>
-<net name="17(TDO)" class="0">
+<net name="D20(TDO)" class="0">
 <segment>
 <wire x1="256.54" y1="205.74" x2="259.08" y2="205.74" width="0.1524" layer="91"/>
@@
 </segment>
 </net>
-<net name="18(TMS)" class="0">
+<net name="D19(TMS)" class="0">
 <segment>
 <wire x1="256.54" y1="203.2" x2="259.08" y2="203.2" width="0.1524" layer="91"/>
@@
 </segment>
 </net>
-<net name="19(TCK)" class="0">
+<net name="D18(TCK)" class="0">
 <segment>
 <wire x1="256.54" y1="200.66" x2="259.08" y2="200.66" width="0.1524" layer="91"/>
 <label x="261.62" y="200.66" size="1.778" layer="95"/>
 <pinref part="IC1" gate="G$1" pin="PCINT18/TCK_PC2"/>
-</segment>
-</net>
-<net name="D23" class="0">
-<segment>
-<wire x1="256.54" y1="193.04" x2="259.08" y2="193.04" width="0.1524" layer="91"/>
-<label x="261.62" y="193.04" size="1.778" layer="95"/>
-<pinref part="IC1" gate="G$1" pin="PCINT31/OC2A_PD7"/>
 </segment>
 </net>
@@
 <junction x="335.28" y="195.58"/>
 </segment>
-<segment>
-<wire x1="195.58" y1="195.58" x2="187.96" y2="195.58" width="0.1524" layer="91"/>
-<label x="185.42" y="195.58" size="1.778" layer="95" rot="MR0"/>
-<pinref part="IC1" gate="G$1" pin="PCINT29/OC1A_PD5"/>
-</segment>
-</net>
-<net name="D6" class="0">
+</net>
+<net name="D2" class="0">
 <segment>
 <wire x1="195.58" y1="236.22" x2="187.96" y2="236.22" width="0.1524" layer="91"/>
@@
 </segment>
 </net>
+<net name="D13" class="0">
+<segment>
+<wire x1="195.58" y1="195.58" x2="187.96" y2="195.58" width="0.1524" layer="91"/>
+<label x="185.42" y="195.58" size="1.778" layer="95" rot="MR0"/>
+<pinref part="IC1" gate="G$1" pin="PCINT29/OC1A_PD5"/>
+</segment>
+</net>
+<net name="D22" class="0">
+<segment>
+<wire x1="256.54" y1="210.82" x2="259.08" y2="210.82" width="0.1524" layer="91"/>
+<label x="261.62" y="210.82" size="1.778" layer="95"/>
+<pinref part="IC1" gate="G$1" pin="PCINT22/TOSC1_PC6"/>
+</segment>
+</net>
+<net name="D23" class="0">
+<segment>
+<wire x1="256.54" y1="213.36" x2="259.08" y2="213.36" width="0.1524" layer="91"/>
+<label x="261.62" y="213.36" size="1.778" layer="95"/>
+<pinref part="IC1" gate="G$1" pin="PCINT23/TOSC2_PC7"/>
+</segment>
+</net>

Commit message: Irškojimai-sprendimai
Relės pakeistos  l293 mikroschema skirta variklių valdymui.
Parts:
- removed C10, C11: 22p, SparkFun:CAPPTH
- removed K1, K2, K3, K4: G5V1, relay-1:G5V1
- removed Y2: 16MHz, SteveMarple:CRYSTAL-RESONATOR
- added C1, C8: 22p, rcl:C-EU025-024X044
- added J11, J12: 6-3.50, con-phoenix-350-1:6-3.50
- added JP1: (no value), pinhead:PINHD-1X16
- added Q1: TIP120V, rocketfarm:TIP120V
- added X2: 16MHz, SparkFun:CRYSTALHC49US
- IC2: value (none) -> L293D; device uln-udn:ULN2803A -> st-microelectronics:L293D
- R7: value 10k -> (none); device SteveMarple:RESISTOR -> resistor-1:R-EU_0309/V
Connections:
- removed net N$47: J105.K, K22.P, K22.P@1
- removed net N$52: J104.K, K22.O
- removed net N$55: J106.K, K22.S
- removed net N$56: J101.K, K12.P, K12.P@1
- removed net N$57: J103.K, K12.O
- removed net N$58: J102.K, K12.S
- removed net N$59: J95.K, K42.P, K42.P@1
- removed net N$60: J94.K, K42.O
- removed net N$61: J96.K, K42.S
- removed net N$62: J92.K, K32.P, K32.P@1
- removed net N$63: J91.K, K32.O
- removed net N$64: J93.K, K32.S
- new net +7V: IC2.VCC2
- new net N$65: J124.K, Q3.C
- new net N$66: J126.K, Q4.C
- new net N$67: J122.K, Q1.C
- new net N$68: C1.2, IC1.XTAL1, X2.1
- new net N$69: C8.2, IC1.XTAL2, X2.2
- new net N$70: IC2.1Y, J62.K
- new net N$71: IC2.2Y, J61.K
- net +5V: now also IC2.1-2EN, IC2.VCC1
- net GND: now also C1.1, C8.1, IC2.GND1, J121.K, J123.K, J125.K, Q1.E; no longer C10.2, C11.2, J41.K, J43.K, Y2.2
- net N$10: now also J114.K, SSR2.DS1; no longer J61.K, SSR2.DS2
- net N$16: now also IC2.1A; no longer C11.1, IC1.XTAL1, Y2.3
- net N$17: now also IC2.2A; no longer C10.1, IC1.XTAL2, Y2.1
- net N$19: now also J113.K, SSR2.DS2; no longer J62.K, SSR2.DS1
- net N$2: now also IC2.4Y, J64.K; no longer IC2.O1, K11.2
- net N$21: now also J112.K, SSR3.DS1; no longer J73.K, SSR3.DS2
- net N$22: now also J111.K, SSR3.DS2; no longer J74.K, SSR3.DS1
- net N$23: now also J16.K, SSR6.DS2; no longer J72.K, SSR4.DS1
- net N$24: now also J15.K, SSR6.DS1; no longer J71.K, SSR4.DS2
- net N$25: now also J14.K, SSR5.DS2; no longer J84.K, SSR5.DS1
- net N$26: now also J13.K, SSR5.DS1; no longer J83.K, SSR5.DS2
- net N$27: now also J12.K, SSR4.DS2; no longer J82.K, SSR6.DS1
- net N$28: now also J11.K, SSR4.DS1; no longer J81.K, SSR6.DS2
- net N$3: now also J63.K; no longer IC2.O2, K21.1
- net N$4: now also IC2.3A; no longer IC2.O3, K31.1
- net N$5: now also IC2.4A; no longer IC2.O4, K41.1
- net N$6: now also J115.K; no longer J63.K
- net N$7: now also Q1.B, R7.2; no longer J42.K, Q4.C
- net N$8: now also R7.1; no longer J44.K, Q3.C
- net N$9: now also J116.K; no longer J64.K
- net VCC: no longer K11.1, K21.2, K31.2, K41.2
Other:
- note added: "DC motor"
- note added: "Enable"
- note added: "Input 1"
- note added: "Input 2"
- note added: "VSS MOTOR SUPPLY"
- note added: "l293d VCC"
- note removed: "Omit load capacitors if resonator"
- note removed: "fitted instead of crystal"
- moved on the sheet: J11, J12, J13, J14, J15, J16, J41, J42, J43, J44, J61, J62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
